Commit message: MoveIt Package is Made! for ROS Melodic and UBUNTU18

File: kuka_description/model/kuka.urdf.xacro (robot description, xacro)
@@ -22,5 +22,5 @@
 			<origin xyz="0 0 0.50" rpy="0 0 0"/>
 			<geometry>
-				<box size="1.0 1.0 1.0"/>
+				<box size="2.0 1.0 1.0"/>
 			</geometry>
 		</visual>
@@ -28,5 +28,5 @@
 			<origin xyz="0 0 0.50" rpy="0 0 0"/>
 			<geometry>
-				<box size="1.0 1.0 1.0"/>
+				<box size="2.0 1.0 1.0"/>
 			</geometry>
 		</collision>

Commit message: a lot of changes regarding the kuka because of the moveit environmental update

File: kuka_description/model/kuka.urdf.xacro (robot description, xacro)
@@ -1,4 +1,4 @@
 <?xml version="1.0"?>
-<robot xmlns:xacro="http://www.ros.org/wiki/xacro" name="single_lwr_robot">
+<robot xmlns:xacro="http://www.ros.org/wiki/xacro" name="KUKA">
 	<!-- Include all models -->
 	<xacro:include filename="$(find kuka_description)/model/kuka_lwr.urdf.xacro"/>
@@ -6,5 +6,5 @@
 	<!-- Attaching My Robot To the WORLD by introducing a dummy link-->
 	<link name="world" />
-    <joint name="world_to_box=" type="fixed">
+    <joint name="world_to_box" type="fixed">
 	  <parent link="world"/>
       <child link="box"/>
@@ -33,5 +33,5 @@
 	</link>
 	<gazebo reference="box">
-		<static>true</static>>
+		<static>true</static>
 	</gazebo>
 	<!-- using the models -->
@@ -39,3 +39,13 @@
 		<origin xyz="0 0 1" rpy="0 0 0"/>
 	</xacro:kuka_lwr>
+			<gazebo>
+			<plugin name="KUKA_lwr_hw_sim" filename="liblwr_hw_gazebo_plugin.so">
+				<robotNamespace></robotNamespace>
+			</plugin>
+		</gazebo>
+		<gazebo>
+		    <plugin name="KUKA_gazebo_ros_control" filename="libgazebo_ros_control.so">
+			    <robotNamespace></robotNamespace>
+			</plugin>
+		</gazebo>
 </robot>

File: kuka_description/model/kuka_lwr.gazebo.xacro (robot description, xacro)
@@ -2,14 +2,4 @@
 <robot xmlns:xacro="http://www.ros.org/wiki/xacro">
 	<xacro:macro name="kuka_lwr_gazebo" params="name">
-		<gazebo>
-			<plugin name="${name}_lwr_hw_sim" filename="liblwr_hw_gazebo_plugin.so">
-				<robotNamespace>${name}</robotNamespace>
-			</plugin>
-		</gazebo>
-		<gazebo>
-		    <plugin name="gazebo_ros_control" filename="libgazebo_ros_control.so">
-			    <robotNamespace>${name}</robotNamespace>
-			</plugin>
-		</gazebo>
 		<gazebo reference="${name}_base_link">
 			<gravity>true</gravity>

File: kuka_description/model/kuka_lwr.transmission.xacro (robot description, xacro)
@@ -1,6 +1,6 @@
 <?xml version="1.0"?>
 <robot xmlns:xacro="http://www.ros.org/wiki/xacro">
-	<xacro:property name="Interface10" value="PositionJointInterface"/>
-	<xacro:property name="Interface30" value="EffortJointInterface"/>
+	<xacro:property name="Interface10" value="hardware_interface/PositionJointInterface"/>
+	<!-- <xacro:property name="Interface30" value="hardware_interface/EffortJointInterface"/> -->
 	<xacro:macro name="kuka_lwr_transmission" params="name">
 		<transmission name="${name}_a1_trans">
@@ -8,5 +8,7 @@
 			<joint name="${name}_a1_joint">
 				<hardwareInterface>${Interface10}</hardwareInterface>
-				<hardwareInterface>${Interface30}</hardwareInterface>
+			    <!--
+			    <hardwareInterface>${Interface30}</hardwareInterface>
+			    -->
 			</joint>
 			<actuator name="${name}_a1_motor">
@@ -18,5 +20,7 @@
 			<joint name="${name}_a2_joint">
 				<hardwareInterface>${Interface10}</hardwareInterface>
+				<!--
 				<hardwareInterface>${Interface30}</hardwareInterface>
+				-->
 			</joint>
 			<actuator name="${name}_a2_motor">
@@ -28,5 +32,7 @@
 			<joint name="${name}_a3_joint">
 				<hardwareInterface>${Interface10}</hardwareInterface>
+				<!--
 				<hardwareInterface>${Interface30}</hardwareInterface>
+				-->
 			</joint>
 			<actuator name="${name}_a3_motor">
@@ -38,5 +44,7 @@
 			<joint name="${name}_a4_joint">
 				<hardwareInterface>${Interface10}</hardwareInterface>
+				<!--
 				<hardwareInterface>${Interface30}</hardwareInterface>
+				-->
 			</joint>
 			<actuator name="${name}_a4_motor">
@@ -48,5 +56,7 @@
 			<joint name="${name}_a5_joint">
 				<hardwareInterface>${Interface10}</hardwareInterface>
+				<!--
 				<hardwareInterface>${Interface30}</hardwareInterface>
+				-->
 			</joint>
 			<actuator name="${name}_a5_motor">
@@ -58,5 +68,7 @@
 			<joint name="${name}_a6_joint">
 				<hardwareInterface>${Interface10}</hardwareInterface>
+				<!--
 				<hardwareInterface>${Interface30}</hardwareInterface>
+				-->
 			</joint>
 			<actuator name="${name}_a6_motor">
@@ -68,5 +80,7 @@
 			<joint name="${name}_a7_joint">
 				<hardwareInterface>${Interface10}</hardwareInterface>
+				<!--
 				<hardwareInterface>${Interface30}</hardwareInterface>
+				-->
 			</joint>
 			<actuator name="${name}_a7_motor">
@@ -78,5 +92,7 @@
 			<joint name="${name}_a8_joint">
 				<hardwareInterface>${Interface10}</hardwareInterface>
+				<!--
 				<hardwareInterface>${Interface30}</hardwareInterface>
+				-->
 			</joint>
 			<actuator name="${name}_a8_motor">
@@ -84,4 +100,75 @@
 			</actuator>
 		</transmission>
+		<!-- Suggested by MoveIt-->
+		    <transmission name="trans_KUKA_a1_joint">
+        <type>transmission_interface/SimpleTransmission</type>
+        <joint name="KUKA_a1_joint">
+            <hardwareInterface>hardware_interface/EffortJointInterface</hardwareInterface>
+        </joint>
+        <actuator name="KUKA_a1_joint_motor">
+            <hardwareInterface>hardware_interface/EffortJointInterface</hardwareInterface>
+            <mechanicalReduction>1</mechanicalReduction>
+        </actuator>
+    </transmission>
+    <transmission name="trans_KUKA_a2_joint">
+        <type>transmission_interface/SimpleTransmission</type>
+        <joint name="KUKA_a2_joint">
+            <hardwareInterface>hardware_interface/EffortJointInterface</hardwareInterface>
+        </joint>
+        <actuator name="KUKA_a2_joint_motor">
+            <hardwareInterface>hardware_interface/EffortJointInterface</hardwareInterface>
+            <mechanicalReduction>1</mechanicalReduction>
+        </actuator>
+    </transmission>
+    <transmission name="trans_KUKA_a3_joint">
+        <type>transmission_interface/SimpleTransmission</type>
+        <joint name="KUKA_a3_joint">
+            <hardwareInterface>hardware_interface/EffortJointInterface</hardwareInterface>
+        </joint>
+        <actuator name="KUKA_a3_joint_motor">
+            <hardwareInterface>hardware_interface/EffortJointInterface</hardwareInterface>
+            <mechanicalReduction>1</mechanicalReduction>
+        </actuator>
+    </transmission>
+    <transmission name="trans_KUKA_a4_joint">
+        <type>transmission_interface/SimpleTransmission</type>
+        <joint name="KUKA_a4_joint">
+            <hardwareInterface>hardware_interface/EffortJointInterface</hardwareInterface>
+        </joint>
+        <actuator name="KUKA_a4_joint_motor">
+            <hardwareInterface>hardware_interface/EffortJointInterface</hardwareInterface>
+            <mechanicalReduction>1</mechanicalReduction>
+        </actuator>
+    </transmission>
+    <transmission name="trans_KUKA_a5_joint">
+        <type>transmission_interface/SimpleTransmission</type>
+        <joint name="KUKA_a5_joint">
+            <hardwareInterface>hardware_interface/EffortJointInterface</hardwareInterface>
+        </joint>
+        <actuator name="KUKA_a5_joint_motor">
+            <hardwareInterface>hardware_interface/EffortJointInterface</hardwareInterface>
+            <mechanicalReduction>1</mechanicalReduction>
+        </actuator>
+    </transmission>
+    <transmission name="trans_KUKA_a6_joint">
+        <type>transmission_interface/SimpleTransmission</type>
+        <joint name="KUKA_a6_joint">
+            <hardwareInterface>hardware_interface/EffortJointInterface</hardwareInterface>
+        </joint>
+        <actuator name="KUKA_a6_joint_motor">
+            <hardwareInterface>hardware_interface/EffortJointInterface</hardwareInterface>
+            <mechanicalReduction>1</mechanicalReduction>
+        </actuator>
+    </transmission>
+    <transmission name="trans_KUKA_a7_joint">
+        <type>transmission_interface/SimpleTransmission</type>
+        <joint name="KUKA_a7_joint">
+            <hardwareInterface>hardware_interface/EffortJointInterface</hardwareInterface>
+        </joint>
+        <actuator name="KUKA_a7_joint_motor">
+            <hardwareInterface>hardware_interface/EffortJointInterface</hardwareInterface>
+            <mechanicalReduction>1</mechanicalReduction>
+        </actuator>
+    </transmission>
 	</xacro:macro>
 </robot>
