Commit message: adding controller and hardware congfiguration

File: kuka_description/model/kuka_lwr.gazebo.xacro (robot description, xacro)
@@ -2,12 +2,14 @@
 <robot xmlns:xacro="http://www.ros.org/wiki/xacro">
 	<xacro:macro name="kuka_lwr_gazebo" params="name">
+<!--
 		<gazebo>
 			<plugin name="KUKA_lwr_hw_sim" filename="liblwr_hw_gazebo_plugin.so">
-				<robotNamespace>KUKA</robotNamespace>
+				<robotNamespace>/KUKA</robotNamespace>
 			</plugin>
 		</gazebo>
+-->
 		<gazebo>
-		    <plugin name="KUKA_gazebo_ros_control" filename="libgazebo_ros_control.so">
-			    <robotNamespace>KUKA</robotNamespace>
+		    <plugin name="gazebo_ros_control" filename="libgazebo_ros_control.so">
+			    <robotNamespace>/KUKA</robotNamespace>
 			</plugin>
 		</gazebo>

File: kuka_description/model/kuka_lwr.transmission.xacro (robot description, xacro)
@@ -1,6 +1,8 @@
 <?xml version="1.0"?>
 <robot xmlns:xacro="http://www.ros.org/wiki/xacro">
-	<xacro:property name="Interface10" value="hardware_interface/PositionJointInterface"/>
-	<!-- <xacro:property name="Interface30" value="hardware_interface/EffortJointInterface"/> -->
+<xacro:property name="Interface10" value="hardware_interface/PositionJointInterface"/>
+	<!--
+			<xacro:property name="Interface30" value="hardware_interface/EffortJointInterface"/>
+    -->
 	<xacro:macro name="kuka_lwr_transmission" params="name">
 		<transmission name="${name}_a1_trans">
@@ -9,5 +11,5 @@
 				<hardwareInterface>${Interface10}</hardwareInterface>
 			    <!--
-			    <hardwareInterface>${Interface30}</hardwareInterface>
+				<hardwareInterface>${Interface30}</hardwareInterface>
 			    -->
 			</joint>
@@ -100,75 +102,4 @@
 			</actuator>
 		</transmission>
-		<!-- Suggested by MoveIt-->
-		    <transmission name="trans_KUKA_a1_joint">
-        <type>transmission_interface/SimpleTransmission</type>
-        <joint name="KUKA_a1_joint">
-            <hardwareInterface>hardware_interface/EffortJointInterface</hardwareInterface>
-        </joint>
-        <actuator name="KUKA_a1_joint_motor">
-            <hardwareInterface>hardware_interface/EffortJointInterface</hardwareInterface>
-            <mechanicalReduction>1</mechanicalReduction>
-        </actuator>
-    </transmission>
-    <transmission name="trans_KUKA_a2_joint">
-        <type>transmission_interface/SimpleTransmission</type>
-        <joint name="KUKA_a2_joint">
-            <hardwareInterface>hardware_interface/EffortJointInterface</hardwareInterface>
-        </joint>
-        <actuator name="KUKA_a2_joint_motor">
-            <hardwareInterface>hardware_interface/EffortJointInterface</hardwareInterface>
-            <mechanicalReduction>1</mechanicalReduction>
-        </actuator>
-    </transmission>
-    <transmission name="trans_KUKA_a3_joint">
-        <type>transmission_interface/SimpleTransmission</type>
-        <joint name="KUKA_a3_joint">
-            <hardwareInterface>hardware_interface/EffortJointInterface</hardwareInterface>
-        </joint>
-        <actuator name="KUKA_a3_joint_motor">
-            <hardwareInterface>hardware_interface/EffortJointInterface</hardwareInterface>
-            <mechanicalReduction>1</mechanicalReduction>
-        </actuator>
-    </transmission>
-    <transmission name="trans_KUKA_a4_joint">
-        <type>transmission_interface/SimpleTransmission</type>
-        <joint name="KUKA_a4_joint">
-            <hardwareInterface>hardware_interface/EffortJointInterface</hardwareInterface>
-        </joint>
-        <actuator name="KUKA_a4_joint_motor">
-            <hardwareInterface>hardware_interface/EffortJointInterface</hardwareInterface>
-            <mechanicalReduction>1</mechanicalReduction>
-        </actuator>
-    </transmission>
-    <transmission name="trans_KUKA_a5_joint">
-        <type>transmission_interface/SimpleTransmission</type>
-        <joint name="KUKA_a5_joint">
-            <hardwareInterface>hardware_interface/EffortJointInterface</hardwareInterface>
-        </joint>
-        <actuator name="KUKA_a5_joint_motor">
-            <hardwareInterface>hardware_interface/EffortJointInterface</hardwareInterface>
-            <mechanicalReduction>1</mechanicalReduction>
-        </actuator>
-    </transmission>
-    <transmission name="trans_KUKA_a6_joint">
-        <type>transmission_interface/SimpleTransmission</type>
-        <joint name="KUKA_a6_joint">
-            <hardwareInterface>hardware_interface/EffortJointInterface</hardwareInterface>
-        </joint>
-        <actuator name="KUKA_a6_joint_motor">
-            <hardwareInterface>hardware_interface/EffortJointInterface</hardwareInterface>
-            <mechanicalReduction>1</mechanicalReduction>
-        </actuator>
-    </transmission>
-    <transmission name="trans_KUKA_a7_joint">
-        <type>transmission_interface/SimpleTransmission</type>
-        <joint name="KUKA_a7_joint">
-            <hardwareInterface>hardware_interface/EffortJointInterface</hardwareInterface>
-        </joint>
-        <actuator name="KUKA_a7_joint_motor">
-            <hardwareInterface>hardware_interface/EffortJointInterface</hardwareInterface>
-            <mechanicalReduction>1</mechanicalReduction>
-        </actuator>
-    </transmission>
 	</xacro:macro>
 </robot>

Commit message: ok... debugging the robot

File: kuka_description/model/kuka_lwr.gazebo.xacro (robot description, xacro)
@@ -2,5 +2,4 @@
 <robot xmlns:xacro="http://www.ros.org/wiki/xacro">
 	<xacro:macro name="kuka_lwr_gazebo" params="name">
-<!--
 		<gazebo>
 			<plugin name="KUKA_lwr_hw_sim" filename="liblwr_hw_gazebo_plugin.so">
@@ -8,5 +7,4 @@
 			</plugin>
 		</gazebo>
--->
 		<gazebo>
 		    <plugin name="gazebo_ros_control" filename="libgazebo_ros_control.so">
@@ -46,8 +44,8 @@
 			<material>Gazebo/DarkGrey</material>
 		</gazebo>
-		<gazebo reference="${name}_8_link">
+		<!--<gazebo reference="${name}_8_link">
 			<gravity>true</gravity>
 			<material>Gazebo/Grey</material>
-		</gazebo>
+		</gazebo>-->
 	</xacro:macro>
 </robot>

File: kuka_description/model/kuka_lwr.transmission.xacro (robot description, xacro)
@@ -90,16 +90,13 @@
 			</actuator>
 		</transmission>
-		<transmission name="${name}_a8_trans">
+		<!--<transmission name="${name}_a8_trans">
 			<type>transmission_interface/SimpleTransmission</type>
 			<joint name="${name}_a8_joint">
 				<hardwareInterface>${Interface10}</hardwareInterface>
-				<!--
-				<hardwareInterface>${Interface30}</hardwareInterface>
-				-->
 			</joint>
 			<actuator name="${name}_a8_motor">
 				<mechanicalReduction>1</mechanicalReduction>
 			</actuator>
-		</transmission>
+		</transmission>-->
 	</xacro:macro>
 </robot>

File: kuka_description/model/kuka_lwr.urdf.xacro (robot description, xacro)
@@ -256,5 +256,5 @@
 		</link>
         <!-- Link 9 -->
-		<link name="${name}_8_link">
+		<!--<link name="${name}_8_link">
 			<inertial>
 				<mass value="${tip_mass}"/>
@@ -275,5 +275,5 @@
 			</geometry>
 			</collision>
-		</link>
+		</link>-->
         <!-- List of Joints -->
 		<!-- Second segment of the arm. Joint along z-axis -->
@@ -411,12 +411,12 @@
 -->
 		<!-- Nineth element of the arm. z-axis -->
-		<joint name="${name}_a8_joint" type="fixed">
+<!-- 		<joint name="${name}_a8_joint" type="fixed">
 			<origin xyz="0 0 0.02" rpy="0 0 0"/>
-			<!--axis xyz="0 0 1"/-->
-			<!--limit effort="38" velocity="${velocity_scale * 184 * M_PI / 180}" /-->
-			<!--dynamics friction="10.0" damping="1.0"/-->
+			<axis xyz="0 0 1"/>
+			<limit effort="38" velocity="${velocity_scale * 184 * M_PI / 180}" />
+			<dynamics friction="10.0" damping="1.0"/>
 			<parent link="${name}_7_link"/>
 			<child link="${name}_8_link"/>
-		</joint>
+		</joint>-->
 <!--
 	<joint name="${name}_a7_joint_stiffness" type="fixed">

Commit message: everything changed

File: kuka_description/model/kuka_lwr.gazebo.xacro (robot description, xacro)
@@ -2,9 +2,11 @@
 <robot xmlns:xacro="http://www.ros.org/wiki/xacro">
 	<xacro:macro name="kuka_lwr_gazebo" params="name">
+<!--
 		<gazebo>
 			<plugin name="KUKA_lwr_hw_sim" filename="liblwr_hw_gazebo_plugin.so">
 				<robotNamespace>/KUKA</robotNamespace>
 			</plugin>
-		</gazebo>
+        </gazebo>
+-->
 		<gazebo>
 		    <plugin name="gazebo_ros_control" filename="libgazebo_ros_control.so">

File: kuka_description/model/kuka_lwr.transmission.xacro (robot description, xacro)
@@ -1,8 +1,6 @@
 <?xml version="1.0"?>
 <robot xmlns:xacro="http://www.ros.org/wiki/xacro">
-<xacro:property name="Interface10" value="hardware_interface/PositionJointInterface"/>
-	<!--
-			<xacro:property name="Interface30" value="hardware_interface/EffortJointInterface"/>
-    -->
+	<xacro:property name="Interface10" value="hardware_interface/PositionJointInterface"/>
+	<xacro:property name="Interface30" value="hardware_interface/EffortJointInterface"/>
 	<xacro:macro name="kuka_lwr_transmission" params="name">
 		<transmission name="${name}_a1_trans">
@@ -10,9 +8,9 @@
 			<joint name="${name}_a1_joint">
 				<hardwareInterface>${Interface10}</hardwareInterface>
-			    <!--
 				<hardwareInterface>${Interface30}</hardwareInterface>
-			    -->
 			</joint>
 			<actuator name="${name}_a1_motor">
+				<hardwareInterface>${Interface10}</hardwareInterface>
+				<hardwareInterface>${Interface30}</hardwareInterface>
 				<mechanicalReduction>1</mechanicalReduction>
 			</actuator>
@@ -22,9 +20,9 @@
 			<joint name="${name}_a2_joint">
 				<hardwareInterface>${Interface10}</hardwareInterface>
-				<!--
 				<hardwareInterface>${Interface30}</hardwareInterface>
-				-->
 			</joint>
 			<actuator name="${name}_a2_motor">
+			    <hardwareInterface>${Interface10}</hardwareInterface>
+				<hardwareInterface>${Interface30}</hardwareInterface>
 				<mechanicalReduction>1</mechanicalReduction>
 			</actuator>
@@ -34,9 +32,9 @@
 			<joint name="${name}_a3_joint">
 				<hardwareInterface>${Interface10}</hardwareInterface>
-				<!--
 				<hardwareInterface>${Interface30}</hardwareInterface>
-				-->
 			</joint>
 			<actuator name="${name}_a3_motor">
+			    <hardwareInterface>${Interface10}</hardwareInterface>
+				<hardwareInterface>${Interface30}</hardwareInterface>
 				<mechanicalReduction>1</mechanicalReduction>
 			</actuator>
@@ -46,9 +44,9 @@
 			<joint name="${name}_a4_joint">
 				<hardwareInterface>${Interface10}</hardwareInterface>
-				<!--
 				<hardwareInterface>${Interface30}</hardwareInterface>
-				-->
 			</joint>
 			<actuator name="${name}_a4_motor">
+			    <hardwareInterface>${Interface10}</hardwareInterface>
+				<hardwareInterface>${Interface30}</hardwareInterface>
 				<mechanicalReduction>1</mechanicalReduction>
 			</actuator>
@@ -58,9 +56,9 @@
 			<joint name="${name}_a5_joint">
 				<hardwareInterface>${Interface10}</hardwareInterface>
-				<!--
 				<hardwareInterface>${Interface30}</hardwareInterface>
-				-->
 			</joint>
 			<actuator name="${name}_a5_motor">
+			    <hardwareInterface>${Interface10}</hardwareInterface>
+				<hardwareInterface>${Interface30}</hardwareInterface>
 				<mechanicalReduction>1</mechanicalReduction>
 			</actuator>
@@ -70,9 +68,9 @@
 			<joint name="${name}_a6_joint">
 				<hardwareInterface>${Interface10}</hardwareInterface>
-				<!--
 				<hardwareInterface>${Interface30}</hardwareInterface>
-				-->
 			</joint>
 			<actuator name="${name}_a6_motor">
+			    <hardwareInterface>${Interface10}</hardwareInterface>
+				<hardwareInterface>${Interface30}</hardwareInterface>
 				<mechanicalReduction>1</mechanicalReduction>
 			</actuator>
@@ -82,21 +80,12 @@
 			<joint name="${name}_a7_joint">
 				<hardwareInterface>${Interface10}</hardwareInterface>
-				<!--
 				<hardwareInterface>${Interface30}</hardwareInterface>
-				-->
 			</joint>
 			<actuator name="${name}_a7_motor">
+			    <hardwareInterface>${Interface10}</hardwareInterface>
+				<hardwareInterface>${Interface30}</hardwareInterface>
 				<mechanicalReduction>1</mechanicalReduction>
 			</actuator>
 		</transmission>
-		<!--<transmission name="${name}_a8_trans">
-			<type>transmission_interface/SimpleTransmission</type>
-			<joint name="${name}_a8_joint">
-				<hardwareInterface>${Interface10}</hardwareInterface>
-			</joint>
-			<actuator name="${name}_a8_motor">
-				<mechanicalReduction>1</mechanicalReduction>
-			</actuator>
-		</transmission>-->
 	</xacro:macro>
 </robot>

File: kuka_description/model/kuka_lwr.urdf.xacro (robot description, xacro)
@@ -11,5 +11,6 @@
 	<xacro:property name="link_mass" value="2.35"/>
     <xacro:property name="wrist_mass" value="1.1"/>
-    <xacro:property name="tip_mass" value="0.25"/>
+    <xacro:property name="tip_mass" value="2.60"/>
+    <!--xacro:property name="tip_mass" value="0.25"/-->
 	<xacro:property name="velocity_scale" value="1"/>
 	<xacro:property name="effort_scale" value="1"/>
@@ -254,4 +255,16 @@
 			</geometry>
 			</collision>
+			<collision>
+			<origin xyz="0 0 0.19" rpy="0 0 0"/>
+			<geometry>
+				<cylinder radius="0.01" length="0.15"/>
+			</geometry>
+			</collision>
+			<collision>
+			<origin xyz="0 0 0.07" rpy="0 0 0"/>
+			<geometry>
+				<cylinder radius="0.045" length="0.105"/>
+			</geometry>
+			</collision>
 		</link>
         <!-- Link 9 -->
